File: panel/attiny-usb_panel.kicad_pcb (KiCad board)
At the start: 2 copper layers, 84.7 x 53.2 mm, 85 parts, among them J2 Conn_01x06, J3 Conn_01x02, J4 Conn_01x06, J5 Conn_01x02, J6 Conn_01x06, J7 Conn_01x02, U1 ATtiny85-20P, U3 ATtiny85-20P, U5 ATtiny85-20P

Commit message: create panel for modified version
Parts:
- removed the C1 at (164.9, 137.4)
- removed the C2 at (148.5, 138.3)
- removed the C3 at (164.9, 119.0)
- removed the C3 at (119.8, 130.0)
- removed the C4 at (136.2, 129.1)
- removed the C4 at (148.5, 120.0)
- removed the C5 at (164.9, 100.6)
- removed the C5 at (119.8, 148.4)
- removed the C6 at (136.2, 147.4)
- removed the C6 at (148.5, 101.5)
- removed the D4 at (115.6, 130.1)
- removed the D5 at (115.6, 118.9)
- removed the D7 at (115.6, 148.5)
- removed the D8 at (115.6, 137.3)
- removed the J4 at (155.2, 130.8)
- removed the J4 at (129.5, 118.2)
- removed the J5 at (160.3, 118.2)
- removed the J5 at (124.4, 130.8)
- removed the J6 at (155.2, 112.5)
- removed the J6 at (129.5, 136.6)
- removed the J7 at (124.4, 149.2)
- removed the J7 at (160.3, 99.8)
- removed the mouse-bite-2mm-slot at (162.7, 115.3)
- removed the mouse-bite-2mm-slot at (162.7, 133.7)
- removed the mouse-bite-2mm-slot at (122.0, 133.7)
- removed the mouse-bite-2mm-slot at (122.0, 115.3)
- added C1: 100n, Capacitor_SMD:C_0805_2012Metric_Pad1.18x1.45mm_HandSolder, F.Cu at (119.8, 130.0)
- added C1: 100n, Capacitor_SMD:C_0805_2012Metric_Pad1.18x1.45mm_HandSolder, F.Cu at (119.8, 148.4)
- added C1: 100n, Capacitor_SMD:C_0805_2012Metric_Pad1.18x1.45mm_HandSolder, F.Cu at (164.9, 137.4)
- added C2: 100n, Capacitor_SMD:C_0805_2012Metric_Pad1.18x1.45mm_HandSolder, F.Cu at (136.2, 147.4)
- added C2: 100n, Capacitor_SMD:C_0805_2012Metric_Pad1.18x1.45mm_HandSolder, F.Cu at (148.5, 138.3)
- added C2: 100n, Capacitor_SMD:C_0805_2012Metric_Pad1.18x1.45mm_HandSolder, F.Cu at (136.2, 129.1)
- added C3: 100n, Capacitor_SMD:C_0805_2012Metric_Pad1.18x1.45mm_HandSolder, F.Cu at (164.9, 119.0)
- added C4: 100n, Capacitor_SMD:C_0805_2012Metric_Pad1.18x1.45mm_HandSolder, F.Cu at (148.5, 120.0)
- added C5: 100n, Capacitor_SMD:C_0805_2012Metric_Pad1.18x1.45mm_HandSolder, F.Cu at (164.9, 100.6)
- added C6: 100n, Capacitor_SMD:C_0805_2012Metric_Pad1.18x1.45mm_HandSolder, F.Cu at (148.5, 101.5)
- added D1: 3V6, Diode_SMD:D_SOD-123, F.Cu at (115.6, 148.5)
- added D1: 3V6, Diode_SMD:D_SOD-123, F.Cu at (115.6, 130.1)
- added D2: 3V6, Diode_SMD:D_SOD-123, F.Cu at (115.6, 137.3)
- added D2: 3V6, Diode_SMD:D_SOD-123, F.Cu at (115.6, 118.9)
- added J1: Conn_01x01, Connector_PinHeader_2.54mm:PinHeader_1x01_P2.54mm_Vertical, F.Cu at (137.1, 102.3)
- added J1: Conn_01x01, Connector_PinHeader_2.54mm:PinHeader_1x01_P2.54mm_Vertical, F.Cu at (147.6, 146.7)
- added J4: Conn_01x01, Connector_PinHeader_2.54mm:PinHeader_1x01_P2.54mm_Vertical, F.Cu at (137.1, 120.7)
- added J4: Conn_01x01, Connector_PinHeader_2.54mm:PinHeader_1x01_P2.54mm_Vertical, F.Cu at (147.6, 128.3)
- added J5: Conn_01x06, Connector_PinHeader_2.54mm:PinHeader_1x06_P2.54mm_Vertical, F.Cu at (155.2, 130.8)
- added J5: Conn_01x06, Connector_PinHeader_2.54mm:PinHeader_1x06_P2.54mm_Vertical, F.Cu at (129.5, 118.2)
- added J6: Conn_01x02, Connector_PinHeader_2.54mm:PinHeader_1x02_P2.54mm_Vertical, F.Cu at (160.3, 118.2)
- added J6: Conn_01x02, Connector_PinHeader_2.54mm:PinHeader_1x02_P2.54mm_Vertical, F.Cu at (124.4, 130.8)
- added J7: Conn_01x01, Connector_PinHeader_2.54mm:PinHeader_1x01_P2.54mm_Vertical, F.Cu at (137.1, 139.1)
- added J7: Conn_01x01, Connector_PinHeader_2.54mm:PinHeader_1x01_P2.54mm_Vertical, F.Cu at (147.6, 109.9)
- added J8: Conn_01x06, Connector_PinHeader_2.54mm:PinHeader_1x06_P2.54mm_Vertical, F.Cu at (129.5, 136.6)
- added J8: Conn_01x06, Connector_PinHeader_2.54mm:PinHeader_1x06_P2.54mm_Vertical, F.Cu at (155.2, 112.5)
- added J9: Conn_01x02, Connector_PinHeader_2.54mm:PinHeader_1x02_P2.54mm_Vertical, F.Cu at (124.4, 149.2)
- added J9: Conn_01x02, Connector_PinHeader_2.54mm:PinHeader_1x02_P2.54mm_Vertical, F.Cu at (160.3, 99.8)
- added mouse-bite-2mm-slot: VAL**, my_lib:mouse-bite-2mm-slot, F.Cu at (118.5, 115.3)
- added mouse-bite-2mm-slot: VAL**, my_lib:mouse-bite-2mm-slot, F.Cu at (118.5, 133.7)
- added mouse-bite-2mm-slot: VAL**, my_lib:mouse-bite-2mm-slot, F.Cu at (166.2, 133.7)
- added mouse-bite-2mm-slot: VAL**, my_lib:mouse-bite-2mm-slot, F.Cu at (166.2, 115.3)
- C1, C2: footprint Capacitor_SMD:C_1206_3216Metric_Pad1.33x1.80mm_HandSolder -> Capacitor_SMD:C_0805_2012Metric_Pad1.18x1.45mm_HandSolder
- D3 (x2), D6 (x2), D9 (x2): value WS2812B -> SK6812
Connections:
- D3 pad 4: unconnected-(D3-DOUT-Pad4) -> Net-(D3-DOUT) (x2)
- D6 pad 4: unconnected-(D3-DOUT-Pad4) -> Net-(D3-DOUT) (x2)
- D9 pad 4: unconnected-(D3-DOUT-Pad4) -> Net-(D3-DOUT) (x2)
Routing:
- net Net-(D3-DOUT): track 0.00 -> 20.6 mm
- net Net-(D3-DIN): track 119.9 -> 102.7 mm
- net +5V: track 429.4 -> 425.3 mm
- net GND: track 87.3 -> 86.3 mm
- net Net-(J2-Pin_6): track 153.3 -> 154.3 mm
Other:
- outline, holes or cut-outs redrawn
